File: assets/circuits/esk8_remote/Esk8_spring_26_2.kicad_sch (KiCad schematic)
At the start: 18 parts, among them J1 Conn_01x02_Pin, J2 Conn_01x05_Pin, U8 NRF-MODULE

Commit message: update circuit schematics
Parts:
- removed #U$7: 18650, symbol Esk8_spring_26-eagle-import:18650
- added BT1: Battery_Cell, symbol Device:Battery_Cell
- J2: footprint Connector_Molex:Molex_KK-396_A-41791-0005_1x05_P3.96mm_Vertical -> Connector_PinHeader_2.54mm:PinHeader_1x05_P2.54mm_Vertical
- U8: footprint NRF24L01:NRF24Lo1 -> (none)
Connections:
- net GND: now also B2.23 (GND@2), BT1.2 (-)
- net at S1.1: now also BT1.1 (+)
- no-connect marks 0 -> 15
Other:
- moved on the sheet: D1, D2, J1, R6, R7
