File: assets/circuits/esk8_remote/Esk8_spring_26.kicad_pcb (KiCad board)
At the start: 2 copper layers, 21.9 x 69 mm, 15 parts, among them J1 Conn_01x02_Pin, J2 Conn_01x05_Pin, U8 NRF-MODULE

Commit message: update circuit schematics
Parts:
- C1, C2: value 100uf -> 100nf
- moved J1 0.50 mm to (155.5, 155.0)
Connections:
- B2 pad 22: (no net) -> unconnected-(B2-RST@2-Pad22)
- B2 pad 23: (no net) -> GND
Routing:
- net GND: track 124.7 -> 132.4 mm
- added copper zone on B.Cu, net GND
- added copper zone on F.Cu, net GND
Other:
- board text added: "+"
- board text added: "-"
- board text added: "E-sk8 controller Josiah Hamm 6/5/26 Colorado School of Mines Labriola Protofund"
- board text added: "GND"
- board text added: "Vraw"

Commit message: delete incorrect base schematic
Parts:
- C1, C2: value 100nf -> 100uf
Changed lines of the file:
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@@
-			)
-		)
-		(property "KiLib_Generator" "resistor/THT"
-			(at 0 0 270)
-			(layer "F.SilkS")
-			(hide yes)
-			(effects
-				(font
-					(size 1 1)
-					(thickness 0.15)
-				)
 			)
 		)
 		(sheetname "/")
-		(sheetfile "Esk8_spring_26_2.kicad_sch")
+		(sheetfile "Esk8_spring_26.kicad_sch")
+		(units
+			(unit
+				(name "A")
+				(pins "1" "2")
+			)
+		)
 		(attr through_hole)
 		(duplicate_pad_numbers_are_jumpers no)
@@
 			)
 		)
-		(property "KiLib_Generator" "connector/pin_header_socket"
-			(at 0 0 90)
-			(layer "F.SilkS")
-			(hide yes)
-			(effects
-				(font
-					(size 1 1)
-					(thickness 0.15)
-				)
-			)
-		)
 		(property ki_fp_filters "Connector*:*_1x??_*")
 		(sheetname "/")
-		(sheetfile "Esk8_spring_26_2.kicad_sch")
+		(sheetfile "Esk8_spring_26.kicad_sch")
+		(units
+			(unit
+				(name "A")
+				(pins "1" "2" "3" "4" "5")
+			)
+		)
 		(attr through_hole)
 		(duplicate_pad_numbers_are_jumpers no)
@@
 			)
 		)
-		(property "KiLib_Generator" "resistor/THT"
-			(at 0 0 270)
-			(layer "F.SilkS")
-			(hide yes)
-			(effects
-				(font
-					(size 1 1)
-					(thickness 0.15)
-				)
-			)
-		)
 		(sheetname "/")
-		(sheetfile "Esk8_spring_26_2.kicad_sch")
+		(sheetfile "Esk8_spring_26.kicad_sch")
+		(units
+			(unit
+				(name "A")
+				(pins "1" "2")
+			)
+		)
 		(attr through_hole)
 		(duplicate_pad_numbers_are_jumpers no)
@@
 			)
 		)
-		(property "KiLib_Generator" "resistor/THT"
-			(at 0 0 180)
-			(layer "F.SilkS")
-			(hide yes)
-			(effects
-				(font
-					(size 1 1)
-					(thickness 0.15)
-				)
-			)
-		)
 		(sheetname "/")
-		(sheetfile "Esk8_spring_26_2.kicad_sch")
+		(sheetfile "Esk8_spring_26.kicad_sch")
+		(units
+			(unit
+				(name "A")
+				(pins "1" "2")
+			)
+		)
 		(attr through_hole)
 		(duplicate_pad_numbers_are_jumpers no)
@@
 			)
 		)
-		(property "KiLib_Generator" "resistor/THT"
-			(at 0 0 180)
-			(layer "F.SilkS")
-			(hide yes)
-			(effects
-				(font
-					(size 1 1)
-					(thickness 0.15)
-				)
-			)
-		)
 		(sheetname "/")
-		(sheetfile "Esk8_spring_26_2.kicad_sch")
+		(sheetfile "Esk8_spring_26.kicad_sch")
+		(units
+			(unit
+				(name "A")
+				(pins "1" "2")
+			)
+		)
 		(attr through_hole)
 		(duplicate_pad_numbers_are_jumpers no)
@@
 		(property ki_fp_filters "Connector*:*_1x??_*")
 		(sheetname "/")
-		(sheetfile "Esk8_spring_26_2.kicad_sch")
+		(sheetfile "Esk8_spring_26.kicad_sch")
+		(units
+			(unit
+				(name "A")
+				(pins "1" "2")
+			)
+		)
 		(attr through_hole)
 		(duplicate_pad_numbers_are_jumpers no)
@@
 			)
 		)
-		(property "Value" "100nf"
+		(property "Value" "100uf"
 			(at 2.5 -0.5 0)
 			(layer "F.SilkS")
@@
 			)
 		)
-		(property "KiLib_Generator" "capacitor/THT/other"
-			(at 0 0 0)
-			(layer "F.SilkS")
-			(hide yes)
-			(effects
-				(font
-					(size 1 1)
-					(thickness 0.15)
-				)
-			)
-		)
 		(property ki_fp_filters "C_*")
 		(sheetname "/")
-		(sheetfile "Esk8_spring_26_2.kicad_sch")
+		(sheetfile "Esk8_spring_26.kicad_sch")
+		(units
+			(unit
+				(name "A")
+				(pins "1" "2")
+			)
+		)
 		(attr through_hole)
 		(duplicate_pad_numbers_are_jumpers no)
@@
 			)
 		)
-		(property "KiLib_Generator" "LED/THT"
-			(at 0 0 90)
-			(layer "F.SilkS")
-			(hide yes)
-			(effects
-				(font
-					(size 1 1)
-					(thickness 0.15)
-				)
-			)
-		)
 		(sheetname "/")
-		(sheetfile "Esk8_spring_26_2.kicad_sch")
+		(sheetfile "Esk8_spring_26.kicad_sch")
+		(units
+			(unit
+				(name "A")
+				(pins "1" "2")
+			)
+		)
 		(attr through_hole)
 		(duplicate_pad_numbers_are_jumpers no)
@@
 			)
 		)
-		(property "KiLib_Generator" "resistor/THT"
-			(at 0 0 180)
-			(layer "F.SilkS")
-			(hide yes)
-			(effects
-				(font
-					(size 1 1)
-					(thickness 0.15)
-				)
-			)
-		)
 		(sheetname "/")
-		(sheetfile "Esk8_spring_26_2.kicad_sch")
+		(sheetfile "Esk8_spring_26.kicad_sch")
+		(units
+			(unit
+				(name "A")
+				(pins "1" "2")
+			)
+		)
 		(attr through_hole)
 		(duplicate_pad_numbers_are_jumpers no)
@@
 			)
 		)
-		(property "KiLib_Generator" "resistor/THT"
-			(at 0 0 0)
-			(layer "F.SilkS")
-			(hide yes)
-			(effects
-				(font
-					(size 1 1)
-					(thickness 0.15)
-				)
-			)
-		)
 		(sheetname "/")
-		(sheetfile "Esk8_spring_26_2.kicad_sch")
+		(sheetfile "Esk8_spring_26.kicad_sch")
+		(units
+			(unit
+				(name "A")
+				(pins "1" "2")
+			)
+		)
 		(attr through_hole)
 		(duplicate_pad_numbers_are_jumpers no)
@@
 			)
 		)
-		(property "KiLib_Generator" "LED/THT"
-			(at 0 0 270)
-			(layer "F.SilkS")
-			(hide yes)
-			(effects
-				(font
-					(size 1 1)
-					(thickness 0.15)
-				)
-			)
-		)
 		(sheetname "/")
-		(sheetfile "Esk8_spring_26_2.kicad_sch")
+		(sheetfile "Esk8_spring_26.kicad_sch")
+		(units
+			(unit
+				(name "A")
+				(pins "1" "2")
+			)
+		)
 		(attr through_hole)
 		(duplicate_pad_numbers_are_jumpers no)
@@
 			)
 		)
-		(property "KiLib_Generator" "resistor/THT"
-			(at 0 0 0)
-			(layer "F.SilkS")
-			(hide yes)
-			(effects
-				(font
-					(size 1 1)
-					(thickness 0.15)
-				)
-			)
-		)
 		(sheetname "/")
-		(sheetfile "Esk8_spring_26_2.kicad_sch")
+		(sheetfile "Esk8_spring_26.kicad_sch")
+		(units
+			(unit
+				(name "A")
+				(pins "1" "2")
+			)
+		)
 		(attr through_hole)
 		(duplicate_pad_numbers_are_jumpers no)
@@
 			)
 		)
-		(property "Value" "100nf"
+		(property "Value" "100uf"
 			(at 2.5 0 180)
 			(layer "F.SilkS")
@@
 			)
 		)
-		(property "KiLib_Generator" "capacitor/THT/other"
-			(at 0 0 180)
-			(layer "F.SilkS")
-			(hide yes)
-			(effects
-				(font
-					(size 1 1)
-					(thickness 0.15)
-				)
-			)
-		)
 		(property ki_fp_filters "C_*")
 		(sheetname "/")
-		(sheetfile "Esk8_spring_26_2.kicad_sch")
+		(sheetfile "Esk8_spring_26.kicad_sch")
+		(units
+			(unit
+				(name "A")
+				(pins "1" "2")
+			)
+		)
 		(attr through_hole)
 		(duplicate_pad_numbers_are_jumpers no)
@@
 		)
 		(sheetname "/")
-		(sheetfile "Esk8_spring_26_2.kicad_sch")
+		(sheetfile "Esk8_spring_26.kicad_sch")
+		(units
+			(unit
+				(name "A")
+				(pins "2" "1" "4" "3" "6" "5" "8" "7")
+			)
+		)
 		(attr smd)
 		(duplicate_pad_numbers_are_jumpers no)
@@
 		)
 		(sheetname "/")
-		(sheetfile "Esk8_spring_26_2.kicad_sch")
+		(sheetfile "Esk8_spring_26.kicad_sch")
+		(units
+			(unit
+				(name "A")
+				(pins "1" "2" "3" "4" "5" "6" "7" "8" "9" "10" "11" "12" "A4" "A5" "24"
+					"23" "22" "21" "20" "19" "18" "17" "16" "15" "14" "13" "A7" "A6"
+				)
+			)
+		)
 		(attr smd)
 		(duplicate_pad_numbers_are_jumpers no)

Commit message: bro I spent 3 hours and changed nothing😭
Parts:
- removed U8: NRF-MODULE, NRF24L01:NRF24Lo1
- added U1: NRF24L01_Breakout, RF_Module:nRF24L01_Breakout, B.Cu at (149.4, 129.8)
- C1, C2: value 100uf -> 100nf
- J1: footprint Connector:JWT_A3963_1x02_P3.96mm_Vertical -> Connector_PinHeader_2.54mm:PinHeader_1x02_P2.54mm_Vertical
- moved R1 10.2 mm to (160.0, 96.5), turned to 180 degrees
- moved R3 10.2 mm to (160.0, 104.0), turned to 180 degrees
- moved R5 10.1 mm to (149.9, 114.6), turned to 0 degrees
- moved R2 10.1 mm to (149.9, 100.5), turned to 0 degrees
- moved R4 10.1 mm to (149.9, 111.5), turned to 0 degrees
- moved J1 4.07 mm to (153.0, 151.8), turned to 0 degrees
- moved D2 3.00 mm to (149.9, 148.0), turned to 90 degrees
- moved D1 2.19 mm to (149.9, 138.8), turned to -90 degrees
- moved R6 0.46 mm to (156.3, 138.4)
- moved R7 0.43 mm to (160.0, 138.4)
- moved C1 0.25 mm to (154.0, 135.3)
Connections:
- net Net-(#U$6-SW) renamed /SW
- net Net-(#U$6-VRX) renamed /VRX
- B2 pad 12: Net-(B2-*9) -> /CE
- B2 pad 13: Net-(B2-*10) -> /CSN
- B2 pad 14: Net-(B2-*11) -> /MOSI
- B2 pad 15: Net-(B2-12) -> /MISO
- B2 pad 16: Net-(B2-13) -> /SCK
- B2 pad 17: Net-(B2-A0) -> /VDIV
- C2 pad 1: Net-(B2-A0) -> /VDIV
- D1 pad 1: Net-(D1-A) -> GND
- D1 pad 2: GND -> Net-(D1-A)
- D2 pad 1: Net-(D2-A) -> GND
- D2 pad 2: GND -> Net-(D2-A)
- R1 pad 1: GND -> Net-(R1-Pad1)
- R1 pad 2: Net-(R1-Pad2) -> GND
- R2 pad 1: Net-(R1-Pad2) -> Net-(R2-Pad1)
- R2 pad 2: Net-(R2-Pad2) -> Net-(R1-Pad1)
- R3 pad 1: Net-(R2-Pad2) -> Net-(R3-Pad1)
- R3 pad 2: Net-(R3-Pad2) -> Net-(R2-Pad1)
- R4 pad 1: Net-(R3-Pad2) -> /VDIV
- R4 pad 2: Net-(B2-A0) -> Net-(R3-Pad1)
- R5 pad 1: Net-(B2-RAW) -> /VDIV
- R5 pad 2: Net-(B2-A0) -> Net-(B2-RAW)
Routing:
- net Net-(B2-*9): track 37.0 -> 0.00 mm
- net /CE: track 0.00 -> 37.0 mm
- net Net-(B2-*11): track 23.2 -> 0.00 mm
- net /MOSI: track 0.00 -> 23.2 mm
- net Net-(B2-13): track 18.7 -> 0.00 mm
- net /SCK: track 0.00 -> 18.7 mm
- net Net-(B2-12): track 17.8 -> 0.00 mm
- net /MISO: track 0.00 -> 17.8 mm
- net Net-(B2-*10): track 12.8 -> 0.00 mm
- net /CSN: track 0.00 -> 12.8 mm
- net Net-(B2-A0): track 11.0 -> 0.00 mm
- net /VDIV: track 0.00 -> 11.0 mm
- net Net-(R3-Pad2): track 7.50 -> 0.00 mm
- net Net-(R3-Pad1): track 0.00 -> 7.50 mm
- net GND: track 132.4 -> 128.3 mm
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Other:
- board size 21.9 x 69 mm -> 21.9 x 68 mm
