File: assets/circuits/esk8_board/recieverBoard.kicad_sch (KiCad schematic)
At the start: 58 parts, among them J2 Conn_01x03_Pin, U2 FLIPSKYVESC, U3 NRF-MODULE

Commit message: first pass at v2 board PCB
Parts:
- added H1, H2, H3: MountingHole, MountingHole:MountingHole_4.3mm_M4, symbol Mechanical:MountingHole
- C2: value C_US -> 140uf
Connections:
- net at U2.2 (B2): no longer #U$1.2 (I2)
